File: Hardware/Aux PCB/MFOS_VCLFO_aux/MFOS_VCLFO_aux.kicad_pcb (KiCad board)
At the start: 2 copper layers, 30 x 84.6 mm, 25 parts, among them J1 Synth_power_2x5, J2 Screw_Terminal_01x03, J3 2 pin Molex header, J7 2 pin Molex header, J8 3 pin Molex header, Q1 J113, U1 TL071

Commit message: Make C4 film, correct dumbass op amp topology
Parts:
- C4: footprint ao_tht:C_Disc_D3.0mm_W1.6mm_P2.50mm -> ao_tht:C_Rect_L7.2mm_W2.5mm_P5.00mm_FKS2_FKP2_MKS2_MKP2
Connections:
- U1 pad 2: Net-(C4-Pad1) -> Net-(R1-Pad2)
- U1 pad 3: Net-(R1-Pad2) -> Net-(C4-Pad1)
Routing:
- net Net-(C4-Pad1): track 25.4 -> 22.9 mm
- net Net-(R1-Pad2): track 18.9 -> 21.4 mm
- net Net-(C4-Pad2): track 9.02 -> 6.52 mm

Commit message: Add some PCB labels
Other:
- board text added: "+"
- board text added: "-"
- board text added: "SYNC"

Commit message: Final revisions before fabrication
Parts:
- removed G***: LOGO, ao_tht:analogoutput_12mm
- removed REF** (x2): MountingHole_3.2mm_M3, MountingHole:MountingHole_3.2mm_M3
- added GRAF1: Graphic, ao_tht:analogoutput_12mm, F.Cu at (111.0, 76.0)
- added GRAF2: Graphic, ao_tht:OSHW-Logo2_7.3x6mm_SilkScreen, F.Cu at (104.0, 132.5)
- added H1: MountingHole, ao_tht:MountingHole_3.2mm_M3, F.Cu at (99.8, 61.8)
- added H2: MountingHole, ao_tht:MountingHole_3.2mm_M3, F.Cu at (99.8, 138.3)
Other:
- board text added: "mod adapted from design by Tim (Servo) Parkhurst CC0 1.0"
- board text removed: "mod adapted from design by Tim (Servo) Parkhurst"
